Commit message: Initial commit

File: docker/pelican.xacro (robot description, xacro)
@@ -20,5 +20,4 @@
   <!-- TODO(ff): Update these params when identifying the model. -->
   <xacro:property name="namespace" value="$(arg namespace)" />
-  <xacro:property name="color" value="$(arg color)" />
   <xacro:property name="rotor_velocity_slowdown_sim" value="10" />
   <xacro:property name="use_mesh_file" value="true" />
@@ -35,5 +34,5 @@
   <xacro:property name="time_constant_up" value="0.0125" /> <!-- [s] -->
   <xacro:property name="time_constant_down" value="0.025" /> <!-- [s] -->
-  <xacro:property name="max_rot_velocity" value="1838" /> <!-- [rad/s] -->
+  <xacro:property name="max_rot_velocity" value="838" /> <!-- [rad/s] -->
   <xacro:property name="rotor_drag_coefficient" value="8.06428e-05" />
   <xacro:property name="rolling_moment_coefficient" value="0.000001" />
@@ -143,51 +142,3 @@
     <xacro:insert_block name="rotor_inertia" />
   </xacro:vertical_rotor>
-  <!-- Macro for the inertia of a cylinder -->
-  <xacro:macro name="cyl_inertia" params="h r mass">
-    <inertia ixx="${0.0833333 * mass * (3*r*r + h*h)}" ixy="0.0" ixz="0.0"
-      iyy="${0.0833333 * mass * (3*r*r + h*h)}" iyz="0.0"
-      izz="${0.5 * mass * (r*r)}" />
-  </xacro:macro>
-<link name="${namespace}/top_rod">
-    <visual>
-      <geometry>
-        <cylinder length="0.12" radius="0.02"/>
-      </geometry>
-    </visual>
-    <collision>
-      <geometry>
-        <cylinder length="0.12" radius="0.05"/>
-      </geometry>
-    </collision>
-    <inertial>
-      <mass value="0.01"/>
-      <xacro:cyl_inertia h="0.12" r="0.05" mass="0.01"/>
-    </inertial>
-</link>
-<joint name="${namespace}/base_to_top_rod" type="fixed">
-  <origin xyz="0 0 0.12" rpy="0 0 0" />
-  <parent link="${namespace}/base_link" />
-  <child link="${namespace}/top_rod" />
-</joint>
-<link name="${namespace}/front_rod">
-    <visual>
-      <geometry>
-        <cylinder length="0.4" radius="0.01"/>
-      </geometry>
-    </visual>
-    <collision>
-      <geometry>
-        <cylinder length="0.4" radius="0.01"/>
-      </geometry>
-    </collision>
-    <inertial>
-      <mass value="0.01"/>
-      <xacro:cyl_inertia h="0.4" r="0.01" mass="0.01"/>
-    </inertial>
-</link>
-<joint name="${namespace}/top_to_front_rod" type="fixed">
-  <origin xyz="0.2 0 0.05" rpy="0 ${pi/2} 0" />
-  <parent link="${namespace}/top_rod" />
-  <child link="${namespace}/front_rod" />
-</joint>
 </robot>
